Commit message: Add standard ROS base frames to URDF

File: URDF/LeKiwi.urdf (robot description, URDF)
Before this commit: robot LeKiwi, 45 links, 44 joints
Links:
- added link base_footprint
- added link base_link
Joints:
- added joint base_footprint_to_base_link: type fixed, parent base_footprint, child base_link, origin xyz=0.0 0.0 0.032937 rpy=0.0 0.0 0.0
- added joint base_link_to_base_plate: type fixed, parent base_link, child base_plate_layer1-v5, origin xyz=0.0 0.0 0.0 rpy=0.0 0.0 -1.5707963267948966

Commit message: Fix reversed shoulder pan axis

File: URDF/LeKiwi.urdf (robot description, URDF)
Before this commit: robot LeKiwi, 45 links, 44 joints
Joints:
- joint STS3215_03a-v1_Revolute-45: axis -3.944304526105059e-31 3.944304526105059e-31 1.0 -> 0.0 0.0 -1.0
